File: PCB/MainPCB/MainPCB.kicad_pcb (KiCad board)
At the start: 2 copper layers, 121.4 x 121.4 mm, 8 parts, among them J1 Conn_01x08_Socket, J2 Conn_01x06_Socket, U1 XB24CDMPIT-001, U2 DEV-16771

Commit message: PCB.  'Tis done.
Parts:
- added ASPD-4525: Conn_01x06_Socket, Connector_PinSocket_2.54mm:PinSocket_1x06_P2.54mm_Vertical, F.Cu at (54.3, 109.4)
- added Buzzer1: Conn_01x02_Pin, Connector_PinHeader_2.54mm:PinHeader_1x02_P2.54mm_Vertical, F.Cu at (45.0, 109.8)
- added C1: 10 uF, Capacitor_SMD:C_1206_3216Metric_Pad1.33x1.80mm_HandSolder, F.Cu at (49.5, 80.9)
- added C2: 100 nF, Capacitor_SMD:C_0402_1005Metric_Pad0.74x0.62mm_HandSolder, F.Cu at (51.4, 87.8)
- added C3: 22 uF, Capacitor_SMD:C_0603_1608Metric_Pad1.08x0.95mm_HandSolder, F.Cu at (58.0, 85.4)
- added C4: 22 uF, Capacitor_SMD:C_0603_1608Metric_Pad1.08x0.95mm_HandSolder, F.Cu at (56.4, 85.4)
- added D1: LED, Connector_PinSocket_2.54mm:PinSocket_1x02_P2.54mm_Vertical, F.Cu at (50.5, 100.6)
- added GPS6MV2: Conn_01x04_Socket, Connector_PinSocket_2.54mm:PinSocket_1x04_P2.54mm_Vertical, F.Cu at (145.8, 83.3)
- added L1: 4.7 uH, Inductor_SMD:L_1008_2520Metric_Pad1.43x2.20mm_HandSolder, F.Cu at (48.4, 87.1)
- added Power1: Conn_01x02_Pin, Connector_PinSocket_2.54mm:PinSocket_1x02_P2.54mm_Vertical, F.Cu at (49.6, 75.5)
- added Q1: NMOS, Package_TO_SOT_THT:TO-220-3_Vertical, F.Cu at (69.1, 97.5)
- added R1: 100 kO, Resistor_SMD:R_0402_1005Metric_Pad0.72x0.64mm_HandSolder, F.Cu at (51.8, 93.1)
- added R2: 1 kO, Resistor_SMD:R_0402_1005Metric_Pad0.72x0.64mm_HandSolder, F.Cu at (47.0, 105.5)
- added R3: 2.1 kO, Resistor_SMD:R_0603_1608Metric_Pad0.98x0.95mm_HandSolder, F.Cu at (69.1, 94.1)
- added SEN291: Conn_01x04_Socket, Connector_PinSocket_2.54mm:PinSocket_1x04_P2.54mm_Vertical, B.Cu at (94.9, 65.6)
- added SW1: SW_DIP_x01, Connector_PinSocket_2.54mm:PinSocket_1x02_P2.54mm_Vertical, F.Cu at (53.3, 78.5)
- added Servo1: Conn_01x03_Pin, Connector_PinHeader_2.54mm:PinHeader_1x03_P2.54mm_Vertical, F.Cu at (47.0, 116.0)
- added Solenoid1: Conn_01x02_Pin, Connector_PinSocket_2.54mm:PinSocket_1x02_P2.54mm_Vertical, F.Cu at (59.3, 100.3)
- added U1: AP63205WU, Package_TO_SOT_SMD:TSOT-23-6, F.Cu at (53.1, 85.5)
- moved TEENSY1 32.2 mm to (112.0, 74.3)
- moved XBEE1 22.2 mm to (88.4, 118.2)
- moved LSM6DSOX+LIS3MDL1 13.6 mm to (93.8, 136.7), turned to -90 degrees
- renumbered J1 to BMP390, J2 to LSM6DSOX+LIS3MDL1, U2 to TEENSY1, U1 to XBEE1
Connections:
- BMP390 pad 4: Net-(J1-Pin_4) -> Net-(ASPD-4525-SCL)
- BMP390 pad 6: Net-(J1-Pin_6) -> Net-(ASPD-4525-SDA)
- LSM6DSOX+LIS3MDL1 pad 4: Net-(J1-Pin_6) -> Net-(ASPD-4525-SCL)
- LSM6DSOX+LIS3MDL1 pad 5: Net-(J1-Pin_4) -> Net-(ASPD-4525-SDA)
- TEENSY1 pad 0: unconnected-(U2-RX1-Pad0) -> Net-(GPS6MV2-TX)
- TEENSY1 pad 1: unconnected-(U2-TX1-Pad1) -> Net-(GPS6MV2-RX)
- TEENSY1 pad 18: Net-(J1-Pin_6) -> Net-(ASPD-4525-SDA)
- TEENSY1 pad 19: Net-(J1-Pin_4) -> Net-(ASPD-4525-SCL)
- TEENSY1 pad 2: unconnected-(U2-OUT2-Pad2) -> Net-(TEENSY1-OUT2)
- TEENSY1 pad 3: unconnected-(U2-LRCLK2-Pad3) -> Net-(Buzzer1-Pin_2)
- TEENSY1 pad 3.3V_1: +5V -> Net-(GPS6MV2-Vcc)
- TEENSY1 pad 3.3V_2: +5V -> Net-(GPS6MV2-Vcc)
- TEENSY1 pad 6: unconnected-(U2-OUT1D-Pad6) -> Net-(Servo1-Pin_3)
- TEENSY1 pad VIN: unconnected-(U2-PadVIN) -> +5V
- XBEE1 pad 1: +5V -> Net-(GPS6MV2-Vcc)
- XBEE1 pad 6: unconnected-(U1-Pad6) -> Net-(GPS6MV2-Vcc)
Routing:
- net GND: track 96.7 -> 338.3 mm, vias 0 -> 1
- net Net-(ASPD-4525-SCL): track 0.00 -> 178.4 mm, vias 0 -> 1
- net Net-(ASPD-4525-SDA): track 0.00 -> 171.4 mm, vias 0 -> 1
- net +5V: track 121.1 -> 251.0 mm, vias 2 -> 1
- net Net-(GPS6MV2-Vcc): track 0.00 -> 95.2 mm
- net Net-(Servo1-Pin_3): track 0.00 -> 92.4 mm
- net Net-(J1-Pin_4): track 91.7 -> 0.00 mm
- net Net-(Buzzer1-Pin_2): track 0.00 -> 89.2 mm
- net Net-(J1-Pin_6): track 89.0 -> 0.00 mm, vias 2 -> 0
- net Net-(GPS6MV2-RX): track 0.00 -> 61.3 mm
- net Net-(GPS6MV2-TX): track 0.00 -> 61.1 mm
- net Net-(TEENSY1-OUT2): track 0.00 -> 56.7 mm
- net Net-(TEENSY1-RX2): track 83.4 -> 53.7 mm
- net Net-(TEENSY1-TX2): track 79.6 -> 53.2 mm
- net Net-(Q1-D): track 0.00 -> 12.0 mm
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Other:
- board text added: "GPS ANTENNA"
- board text removed: "BMP390"
